Commit message: Axis changes urdf

File: URDF/manipulator_m3_v2/urdf/manipulator_m3_v2.urdf (robot description, URDF)
Before this commit: robot manipulator_m3_v2, 4 links, 3 joints
Joints:
- joint J_1: axis 1 0 0 -> 0 0 -1; origin xyz=0 -0.135 0 rpy=1.6861 0 1.5708 -> xyz=0 0 0.135 rpy=0 0 0; type revolute -> continuous
- joint J_2: axis 1 0 0 -> 0.99986 0.017021 0; origin xyz=-0.12 0 0 rpy=-2.4655 0 -1.5708 -> xyz=0 0 0.12 rpy=0 0 -0.13235; type revolute -> continuous
- joint J_3: axis 1 0 0 -> 0.99986 0.017021 0; origin xyz=0 0.25 0 rpy=0.44871 0 0 -> xyz=0.0026628 -0.15642 0.195 rpy=0 0 0; type revolute -> continuous
